Commit message: trying to make controller_manager to work

File: src/car_description/urdf/car_ros2_control.xacro (robot description, xacro)
@@ -10,4 +10,19 @@
             <plugin>gz_ros2_control/GazeboSimSystem</plugin>
         </xacro:unless>
+        <joint name="base_joint" type="fixed">
+            <state_interface name="position"/>
+        </joint>
+        <joint name="steering_joint_fr" type="continuous">
+            <state_interface name="position"/>
+        </joint>
+        <joint name="FR_wheel_joint" type="continuous">
+            <state_interface name="position"/>
+        </joint>
+        <joint name="steering_joint_fl" type="continuous">
+            <state_interface name="position"/>
+        </joint>
+        <joint name="FL_wheel_joint" type="continuous">
+            <state_interface name="position"/>
+        </joint>
         <joint name="RR_wheel_joint" type="continuous">
             <command_interface name="velocity">
@@ -15,5 +30,5 @@
                 <param name="min">100</param>
             </command_interface>
-            <state_interface name="position"/>
+            <state_interface name="position"></state_interface>
             <state_interface name="velocity"/>
         </joint>
