Commit message: trying to implement ackermann controller plugin

File: src/car_description/urdf/car_gazebo.xacro (robot description, xacro)
@@ -49,3 +49,14 @@
         </xacro:unless>
     </gazebo>
+    <gazebo>
+        <plugin filename="ignition-gazebo-joint-state-publisher-system" name="ignition::gazebo::systems::JointStatePublisher">
+            <topic>joint_states</topic>
+            <joint>steering_joint_fr</joint>
+            <joint>steering_joint_fl</joint>
+            <joint>FR_wheel_joint</joint>
+            <joint>FL_wheel_joint</joint>
+            <joint>RR_wheel_joint</joint>
+            <joint>RL_wheel_joint</joint>
+        </plugin>
+    </gazebo>
 </robot>

File: src/car_description/urdf/car_ros2_control.xacro (robot description, xacro)
@@ -10,23 +10,26 @@
             <plugin>gz_ros2_control/GazeboSimSystem</plugin>
         </xacro:unless>
-        <joint name="base_joint" type="fixed">
+        <joint name="steering_joint_fr" type="continuous">
+            <command_interface name="position"/>
             <state_interface name="position"/>
         </joint>
-        <joint name="steering_joint_fr" type="continuous">
-            <state_interface name="position"/>
-        </joint>
+        <!--
         <joint name="FR_wheel_joint" type="continuous">
             <state_interface name="position"/>
         </joint>
+        -->
         <joint name="steering_joint_fl" type="continuous">
+            <command_interface name="position"/>
             <state_interface name="position"/>
         </joint>
+        <!--
         <joint name="FL_wheel_joint" type="continuous">
             <state_interface name="position"/>
         </joint>
+        -->
         <joint name="RR_wheel_joint" type="continuous">
             <command_interface name="velocity">
                 <param name="min">-10</param>
-                <param name="min">100</param>
+                <param name="max">100</param>
             </command_interface>
             <state_interface name="position"></state_interface>
@@ -36,5 +39,5 @@
             <command_interface name="velocity">
                 <param name="min">-10</param>
-                <param name="min">100</param>
+                <param name="max">100</param>
             </command_interface>
             <state_interface name="position"/>

File: src/car_description/urdf/car_urdf.xacro (robot description, xacro)
@@ -28,5 +28,5 @@
             </geometry>
             <material name="red">
-                <color rgba="1.0 0.0 0.0 0.7"/>
+                <color rgba="1.0 0.0 0.0 0.8"/>
             </material>
         </visual>

Commit message: changed pysical simulation values in xacro files

File: src/car_description/urdf/car_gazebo.xacro (robot description, xacro)
@@ -1,39 +1,58 @@
 <?xml version="1.0"?>
 <robot name="car" xmlns:xacro="http://www.ros.org/wiki/xacro">
+    <gazebo reference="base_link">
+        <pose>0 0 0 0 0 0</pose>
+    </gazebo>
     <gazebo reference="FR_wheel">
-        <mu1>1.0E14</mu1>
-        <mu2>1.0E14</mu2>
-        <kp>1.0E12</kp>
+        <mu1>1.0</mu1>
+        <mu2>1.0</mu2>
+        <kp>100000.0</kp>
         <kd>10.0</kd>
-        <minDepth>0.01</minDepth>
+        <minDepth>0.001</minDepth>
         <maxVel>10</maxVel>
         <fDir1>1 0 0</fDir1>
     </gazebo>
     <gazebo reference="FL_wheel">
-        <mu1>1.0E14</mu1>
-        <mu2>1.0E14</mu2>
-        <kp>1.0E12</kp>
+        <mu1>1.0</mu1>
+        <mu2>1.0</mu2>
+        <kp>100000.0</kp>
         <kd>10.0</kd>
-        <minDepth>0.01</minDepth>
+        <minDepth>0.001</minDepth>
         <maxVel>10</maxVel>
         <fDir1>1 0 0</fDir1>
     </gazebo>
     <gazebo reference="RR_wheel">
-        <mu1>1.0E14</mu1>
-        <mu2>1.0E14</mu2>
-        <kp>1.0E12</kp>
+        <mu1>1.0</mu1>
+        <mu2>1.0</mu2>
+        <kp>100000.0</kp>
         <kd>10.0</kd>
-        <minDepth>0.01</minDepth>
+        <minDepth>0.001</minDepth>
         <maxVel>10</maxVel>
         <fDir1>1 0 0</fDir1>
     </gazebo>
+    <gazebo reference="RR_wheel_joint">
+        <velocity>0.0</velocity> <!-- initial velocity -->
+        <damping>0.5</damping> <!-- helps stability -->
+        <maxVel>10.0</maxVel> <!-- limit -->
+        <minDepth>0.01</minDepth>
+        <mu1>1.0</mu1>
+        <mu2>1.0</mu2>
+    </gazebo>
     <gazebo reference="RL_wheel">
-        <mu1>1.0E14</mu1>
-        <mu2>1.0E14</mu2>
-        <kp>1.0E12</kp>
+        <mu1>1.0</mu1>
+        <mu2>1.0</mu2>
+        <kp>100000.0</kp>
         <kd>10.0</kd>
-        <minDepth>0.01</minDepth>
+        <minDepth>0.001</minDepth>
         <maxVel>10</maxVel>
         <fDir1>1 0 0</fDir1>
+    </gazebo>
+    <gazebo reference="RL_wheel_joint">
+        <velocity>0.0</velocity> <!-- initial velocity -->
+        <damping>0.5</damping> <!-- helps stability -->
+        <maxVel>10.0</maxVel> <!-- limit -->
+        <minDepth>0.01</minDepth>
+        <mu1>1.0</mu1>
+        <mu2>1.0</mu2>
     </gazebo>
     <gazebo>

File: src/car_description/urdf/car_ros2_control.xacro (robot description, xacro)
@@ -13,4 +13,6 @@
             <command_interface name="position"/>
             <state_interface name="position"/>
+            <state_interface name="velocity"/>
+            <state_interface name="effort"/>
         </joint>
         <!--
@@ -22,4 +24,6 @@
             <command_interface name="position"/>
             <state_interface name="position"/>
+            <state_interface name="velocity"/>
+            <state_interface name="effort"/>
         </joint>
         <!--
@@ -29,12 +33,14 @@
         -->
         <joint name="RR_wheel_joint" type="continuous">
-            <command_interface name="velocity"></command_interface>
-            <state_interface name="position"></state_interface>
+            <command_interface name="velocity"/>
+            <state_interface name="position"/>
             <state_interface name="velocity"/>
+            <state_interface name="effort"/>
         </joint>
         <joint name="RL_wheel_joint" type="continuous">
-            <command_interface name="velocity"></command_interface>
+            <command_interface name="velocity"/>
             <state_interface name="position"/>
             <state_interface name="velocity"/>
+            <state_interface name="effort"/>
         </joint>
     </ros2_control>

File: src/car_description/urdf/car_urdf.xacro (robot description, xacro)
@@ -73,10 +73,10 @@
             value="20" />
         <inertia
-            ixx="1.3014"
-            ixy="-2.1717E-12"
-            ixz="-1.7928E-12"
-            iyy="0.84577"
-            iyz="-6.4305E-12"
-            izz="0.84577" />
+            ixx="0.2"
+            ixy="0.0"
+            ixz="0.0"
+            iyy="0.4"
+            iyz="0.0"
+            izz="0.4" />
         </inertial>
         <visual>
@@ -132,10 +132,10 @@
                 value="20" />
             <inertia
-                ixx="1.3014"
-                ixy="-2.1717E-12"
-                ixz="-1.7928E-12"
-                iyy="0.84577"
-                iyz="-6.4305E-12"
-                izz="0.84577" />
+            ixx="0.2"
+            ixy="0.0"
+            ixz="0.0"
+            iyy="0.4"
+            iyz="0.0"
+            izz="0.4" />
         </inertial>
         <visual>
@@ -168,11 +168,11 @@
             <mass
                 value="20" />
-            <inertia
-                ixx="1.3014"
-                ixy="-2.1717E-12"
-                ixz="-1.7928E-12"
-                iyy="0.84577"
-                iyz="-6.4305E-12"
-                izz="0.84577" />
+             <inertia
+            ixx="0.2"
+            ixy="0.0"
+            ixz="0.0"
+            iyy="0.4"
+            iyz="0.0"
+            izz="0.4" />
         </inertial>
         <visual>
@@ -198,4 +198,14 @@
         <origin xyz="-1.05 -0.6 -0.5" rpy="0.0 0.0 0.0"/>
     </joint>
+    <transmission name="RR_wheel_trans">
+        <type>transmission_interface/SimpleTransmission</type>
+        <joint name="RR_wheel_joint">
+            <hardwareInterface>velocity</hardwareInterface>
+        </joint>
+        <actuator name="RR_wheel_motor">
+            <hardwareInterface>velocity</hardwareInterface>
+            <mechanicalReduction>1</mechanicalReduction>
+        </actuator>
+    </transmission>
     <link name="RL_wheel">
         <inertial>
@@ -205,11 +215,11 @@
             <mass
                 value="20" />
-            <inertia
-                ixx="1.3014"
-                ixy="-2.1717E-12"
-                ixz="-1.7928E-12"
-                iyy="0.84577"
-                iyz="-6.4305E-12"
-                izz="0.84577" />
+             <inertia
+            ixx="0.2"
+            ixy="0.0"
+            ixz="0.0"
+            iyy="0.4"
+            iyz="0.0"
+            izz="0.4" />
         </inertial>
         <visual>
@@ -235,3 +245,13 @@
         <origin xyz="-1.05 0.6 -0.5" rpy="0.0 0.0 0.0"/>
     </joint>
+    <transmission name="RL_wheel_trans">
+        <type>transmission_interface/SimpleTransmission</type>
+        <joint name="RL_wheel_joint">
+            <hardwareInterface>velocity</hardwareInterface>
+        </joint>
+        <actuator name="RL_wheel_motor">
+            <hardwareInterface>velocity</hardwareInterface>
+            <mechanicalReduction>1</mechanicalReduction>
+        </actuator>
+    </transmission>
 </robot>

Commit message: added mock joints for the ackerman 'rear' wheels. both ackermann and velocity controllers are implemented- need to write a node to use them both

File: src/car_description/urdf/car_gazebo.xacro (robot description, xacro)
@@ -25,11 +25,11 @@
     </gazebo>
     <gazebo reference="RR_wheel">
-        <mu1>1.0</mu1>
-        <mu2>1.0</mu2>
+        <mu1>10.0</mu1>
+        <mu2>10.0</mu2>
         <kp>100000.0</kp>
         <kd>10.0</kd>
         <minDepth>0.001</minDepth>
         <maxVel>10</maxVel>
-        <fDir1>1 0 0</fDir1>
+        <fDir1>1 1 1</fDir1>
     </gazebo>
     <gazebo reference="RR_wheel_joint">
@@ -42,11 +42,11 @@
     </gazebo>
     <gazebo reference="RL_wheel">
-        <mu1>1.0</mu1>
-        <mu2>1.0</mu2>
+        <mu1>10.0</mu1>
+        <mu2>10.0</mu2>
         <kp>100000.0</kp>
         <kd>10.0</kd>
         <minDepth>0.001</minDepth>
         <maxVel>10</maxVel>
-        <fDir1>1 0 0</fDir1>
+        <fDir1>1 1 1</fDir1>
     </gazebo>
     <gazebo reference="RL_wheel_joint">

File: src/car_description/urdf/car_ros2_control.xacro (robot description, xacro)
@@ -18,4 +18,6 @@
         <joint name="FR_wheel_joint" type="continuous">
             <state_interface name="position"/>
+            <state_interface name="velocity"/>
+            <state_interface name="effort"/>
         </joint>
         <joint name="steering_joint_fl" type="continuous">
@@ -27,4 +29,6 @@
         <joint name="FL_wheel_joint" type="continuous">
             <state_interface name="position"/>
+            <state_interface name="velocity"/>
+            <state_interface name="effort"/>
         </joint>
         <joint name="RR_wheel_joint" type="continuous">
@@ -40,4 +44,16 @@
             <state_interface name="effort"/>
         </joint>
+        <joint name="ack_fl_joint" type="continuous">
+            <command_interface name="velocity"/>
+            <state_interface name="position"/>
+            <state_interface name="velocity"/>
+            <state_interface name="effort"/>
+        </joint>
+        <joint name="ack_fr_joint" type="continuous">
+            <command_interface name="velocity"/>
+            <state_interface name="position"/>
+            <state_interface name="velocity"/>
+            <state_interface name="effort"/>
+        </joint>
     </ros2_control>
 </robot>

File: src/car_description/urdf/car_urdf.xacro (robot description, xacro)
@@ -255,3 +255,67 @@
         </actuator>
     </transmission>
+    <link name="ack_fr">
+        <inertial>
+            <origin
+                xyz="0 0 0"
+                rpy="0 0 0" />
+            <mass
+                value="0.001" />
+            <inertia
+                ixx="0.1"
+                ixy="0.0"
+                ixz="0.0"
+                iyy="0.1"
+                iyz="0.0"
+                izz="0.1" />
+        </inertial>
+    </link>
+    <joint name="ack_fr_joint" type="continuous">
+        <parent link="base_link"/>
+        <child link="ack_fr"/>
+        <axis xyz="0.0 1.0 0.0"/>
+        <origin xyz="0.5 -0.6 -0.5" rpy="0.0 0.0 0.0"/>
+    </joint>
+    <transmission name="ack_fr_trans">
+        <type>transmission_interface/SimpleTransmission</type>
+        <joint name="ack_fr_joint">
+            <hardwareInterface>VelocityJointInterface</hardwareInterface>
+        </joint>
+        <actuator name="FR_wheel_motor">
+            <hardwareInterface>VelocityJointInterface</hardwareInterface>
+            <mechanicalReduction>1</mechanicalReduction>
+        </actuator>
+    </transmission>
+    <link name="ack_fl">
+        <inertial>
+            <origin
+                xyz="0 0 0"
+                rpy="0 0 0" />
+            <mass
+                value="0.001" />
+            <inertia
+                ixx="0.1"
+                ixy="0.0"
+                ixz="0.0"
+                iyy="0.1"
+                iyz="0.0"
+                izz="0.1" />
+        </inertial>
+    </link>
+    <joint name="ack_fl_joint" type="continuous">
+        <parent link="base_link"/>
+        <child link="ack_fl"/>
+        <axis xyz="0.0 1.0 0.0"/>
+        <origin xyz="0.5 0.6 -0.5" rpy="0.0 0.0 0.0"/>
+    </joint>
+    <transmission name="ack_fl_trans">
+        <type>transmission_interface/SimpleTransmission</type>
+        <joint name="ack_fl_joint">
+            <hardwareInterface>VelocityJointInterface</hardwareInterface>
+        </joint>
+        <actuator name="FL_wheel_motor">
+            <hardwareInterface>VelocityJointInterface</hardwareInterface>
+            <mechanicalReduction>1</mechanicalReduction>
+        </actuator>
+    </transmission>
 </robot>

Commit message: added ego controller node to control the robot iva the /vel_cmd topic

File: src/car_description/urdf/car_gazebo.xacro (robot description, xacro)
@@ -73,4 +73,5 @@
         <plugin filename="ignition-gazebo-joint-state-publisher-system" name="ignition::gazebo::systems::JointStatePublisher">
             <topic>joint_states</topic>
+            <joint>base_joint</joint>
             <joint>steering_joint_fr</joint>
             <joint>steering_joint_fl</joint>
