Commit message: new ego body

File: src/car_description/urdf/car_urdf.xacro (robot description, xacro)
@@ -23,7 +23,7 @@
         </inertial>
         <visual>
-            <origin rpy="1.57 0 -1.57" xyz= "1.5 0.75 -0.5"/>
-            <geometry>
-                <mesh filename="package://car_description/meshes/polygon_car.STL"/>
+            <origin rpy="1.57 0 -1.57" xyz= "1.5 0.917885 -0.5"/>
+            <geometry>
+                <mesh filename="package://car_description/meshes/ego_cyber.STL"/>
             </geometry>
             <material name="red">
@@ -32,7 +32,7 @@
         </visual>
         <collision>
-            <origin rpy="1.57 0 -1.57" xyz= "1.5 0.75 -0.5"/>
-            <geometry>
-                <mesh filename="package://car_description/meshes/polygon_car.STL"/>
+            <origin rpy="1.57 0 -1.57" xyz= "1.5 0.917885 -0.5"/>
+            <geometry>
+                <mesh filename="package://car_description/meshes/ego_cyber.STL"/>
             </geometry>
         </collision>
